Commit message: Implement task 4 URDF robot model

File: ros2_ws/src/exam_robot/urdf/exam_robot.urdf (robot description, URDF)
Before this commit: robot exam_robot, 2 links, 1 joints
Links:
- added link left_wheel; visual cylinder length=0.04 radius=0.08
- added link right_wheel; visual cylinder length=0.04 radius=0.08
- link base_link: geometry visual box size=0.4 0.3 0.1
- link sensor_link: geometry visual box size=0.05 0.05 0.05
Joints:
- added joint left_wheel_joint: type continuous, parent base_link, child left_wheel, origin xyz=0 0.17 0 rpy=0 0 0, axis 0 0 1
- added joint right_wheel_joint: type continuous, parent base_link, child right_wheel, origin xyz=0 -0.17 0 rpy=0 0 0, axis 0 0 1
- joint sensor_joint: origin xyz=0.15 0.0 0.10 rpy=0 0 0 -> xyz=0.2 0.0 0.08 rpy=0 0 0
